Commit message: Modify some link masses

File: xacro/edu/fingeredu_macro.xacro (robot description, xacro)
@@ -72,5 +72,5 @@
                 <!-- CoM is only estimated based -->
                 <origin rpy="0 0 0" xyz="-0.079 0 0"/>
-                <mass value="0.14854"/>
+                <mass value="0.157"/>
                 <inertia izz="0.00041" iyz="0.00000" ixz="0.00000"
                                        iyy="0.00041" ixy="0.00005"
@@ -86,5 +86,5 @@
             <inertial>
                 <origin rpy="0 0 0" xyz="0 -0.019 -0.079"/>
-                <mass value="0.14854"/>
+                <mass value="0.16"/>
                 <inertia ixx="0.00041" ixy="0.00000" ixz="0.00000"
                                        iyy="0.00041" iyz="0.00005"
@@ -103,5 +103,5 @@
             <inertial>
                 <origin rpy="0 0 0" xyz="0 -0.009 -0.089"/>
-                <mass value="0.03070"/>
+                <mass value="0.035"/>
                 <inertia ixx="0.00012" ixy="0.00000" ixz="0.00000"
                                        iyy="0.00012" iyz="0.00000"
@@ -128,5 +128,5 @@
             <parent link="finger_base_link${suffix}"/>
             <child link="finger_upper_link${suffix}"/>
-            <limit effort="1000" lower="-${pi/2}" upper="${pi/2}" velocity="1000"/>
+            <limit effort="0.36" lower="-${pi/2}" upper="${pi/2}" velocity="20"/>
             <axis xyz="-1 0 0"/>
             <origin rpy="0 0 0" xyz="0 0 0"/>
@@ -135,5 +135,5 @@
             <parent link="finger_upper_link${suffix}"/>
             <child link="finger_middle_link${suffix}"/>
-            <limit effort="1000" lower="-${pi/2}" upper="${pi/2}" velocity="1000"/>
+            <limit effort="0.36" lower="-${pi/2}" upper="${pi/2}" velocity="20"/>
             <axis xyz="0 1 0"/>
             <origin rpy="0 0 0" xyz="0 -0.014 0"/>
@@ -142,5 +142,5 @@
             <parent link="finger_middle_link${suffix}"/>
             <child link="finger_lower_link${suffix}"/>
-            <limit effort="1000" lower="-${pi}" upper="${pi}" velocity="1000"/>
+            <limit effort="0.36" lower="-${pi}" upper="${pi}" velocity="20"/>
             <axis xyz="0 1 0"/>
             <origin rpy="0 0 0" xyz="0 -0.03745 -0.16"/>

File: xacro/edu/trifingeredu.urdf.xacro (robot description, xacro)
@@ -4,5 +4,5 @@
     <xacro:include filename="fingeredu_macro.xacro" />
     <xacro:include filename="../macros.xacro" />
-    <xacro:property name="distance_to_ground" value="${0.363 - 0.08}" />
+    <xacro:property name="distance_to_ground" value="${0.362 - 0.08}" />
     <xacro:property name="distance_to_center" value="-${offset_x_base_to_front + 0.02}" />
     <xacro:property name="angle_0" value="${radians(0)}"/>
